Commit message: Add files via upload

File: rmp01_bot_description/urdf/rmp01_bot.xacro (robot description, xacro)
@@ -108,5 +108,5 @@
   <parent link="base_link"/>
   <child link="right_wheel_1"/>
-  <axis xyz="0.0 -1.0 0.0"/>
+  <axis xyz="0.0 1.0 0.0"/>
 </joint>
 <joint name="left_wheel_joint" type="continuous">
@@ -116,10 +116,10 @@
   <axis xyz="0.0 1.0 0.0"/>
 </joint>
-<joint name="Rigid 3" type="fixed">
+<joint name="caster_joint" type="fixed">
   <origin xyz="0.1 0.0 0.025" rpy="0 0 0"/>
   <parent link="base_link"/>
   <child link="caster_1"/>
 </joint>
-<joint name="Rigid 4" type="fixed">
+<joint name="lidar_joint" type="fixed">
   <origin xyz="0.0 0.0 0.08" rpy="0 0 0"/>
   <parent link="base_link"/>
